File: hardware/prj-kicad/cowkeyr-sc-g0.kicad_sch (KiCad schematic)
At the start: 0 parts

Commit message: HW: Insert SmartCard connector (sch + footprint)
Parts:
- added C10: 1uF, cowkeyr-sc-g0:SMD0603, symbol cowkeyr-sc-g0:C
- added P2: CONN_SC, cowkeyr-sc-g0:CONN_7312P0225AxxLF, symbol cowkeyr-sc-g0:CONN_SC
- added R10: 10k, cowkeyr-sc-g0:SMD0603, symbol cowkeyr-sc-g0:R
- added TP_SC0, TP_SC1, TP_SC2, TP_SC3, TP_SC4, TP_SC5, TP_SC6, TP_SC7, TP_SC8: CONN_1, cowkeyr-sc-g0:TP_PIN, symbol cowkeyr-sc-g0:CONN_1
Connections:
- new net +3.3V: R10.2
- new net +V_SC: C10.1, P2.C1 (VCC), TP_SC1.1
- new net GND: C10.2, P2.2, P2.C5 (GND), TP_SC5.1
- new net SC_C4: P2.C4, TP_SC4.1
- new net SC_C6: P2.C6 (VPP), TP_SC6.1
- new net SC_C8: P2.C8, TP_SC8.1
- new net SC_CLK: P2.C3 (CLK), TP_SC3.1
- new net SC_DETECT: P2.1, R10.1, TP_SC0.1
- new net SC_IO: P2.C7 (IO), TP_SC7.1
- new net SC_RST: P2.C2 (RST), TP_SC2.1

Commit message: HW: Replace smartcard connector (bad size) and add power supplies
Parts:
- added C12, C13, C8, C9: 4,7uF, cowkeyr-sc-g0:SMD0603, symbol cowkeyr-sc-g0:C
- added C3, C5: 10uF, cowkeyr-sc-g0:SMD0805, symbol cowkeyr-sc-g0:C
- added C4: 100nF, cowkeyr-sc-g0:SMD0603, symbol cowkeyr-sc-g0:C
- added C6: 470pF, cowkeyr-sc-g0:SMD0603, symbol cowkeyr-sc-g0:C
- added C7: n/a, cowkeyr-sc-g0:SMD1210, symbol cowkeyr-sc-g0:C
- added L1, L2: 2,2uH, cowkeyr-sc-g0:I_CDRH2D14, symbol cowkeyr-sc-g0:INDUCTOR
- added P1: CONN_USB-C, cowkeyr-sc-g0:CONN_632723300011, symbol cowkeyr-sc-g0:CONN_USB-C
- added R11, R15: 10k, cowkeyr-sc-g0:SMD0603, symbol cowkeyr-sc-g0:R
- added R12: 422k, cowkeyr-sc-g0:SMD0603, symbol cowkeyr-sc-g0:R
- added R13: 75k, cowkeyr-sc-g0:SMD0603, symbol cowkeyr-sc-g0:R
- added R14: 47k, cowkeyr-sc-g0:SMD0603, symbol cowkeyr-sc-g0:R
- added U2, U3: LM3671, cowkeyr-sc-g0:SOT23-5, symbol cowkeyr-sc-g0:LM3671
- added U4, U5, U6: SN74LVC1T45, cowkeyr-sc-g0:SOT23-6, symbol cowkeyr-sc-g0:SN74LVC1T45
- added U9: SN74LVC1G3157, cowkeyr-sc-g0:SOT23-6, symbol cowkeyr-sc-g0:SN74LVC1G3157
- P2: footprint cowkeyr-sc-g0:CONN_7312P0225AxxLF -> cowkeyr-sc-g0:CONN_CCM01-25xx
Connections:
- net +3.3V: now also C7.1, C8.1, C9.1, L1.2, U2.4 (FB), U4.1 (VCCA), U4.5 (DIR), U5.1 (VCCA), U5.5 (DIR), U6.1 (VCCA), U9.5
- net +V_SC: now also C12.1, C13.1, L2.2, R12.1, U4.6 (VCCB), U5.6 (VCCB), U6.6 (VCCB)
- net GND: now also P2.0, C12.2, C13.2, C3.2, C4.2, C5.2, C6.2, C7.2, C8.2, C9.2, P1.A1, P1.A12, P1.B1, P1.B12, P1.SHLD, R11.2, R13.2, R14.2, R15.2, U2.2, U3.2, U4.2, U5.2, U6.2, U9.2
- net SC_CLK: now also U5.3 (A); no longer P2.C3 (CLK), TP_SC3.1
- net SC_IO: now also U6.3 (A); no longer P2.C7 (IO), TP_SC7.1
- net SC_RST: now also U4.3 (A); no longer P2.C2 (RST), TP_SC2.1
- new net: R14.1, U9.1 (B2)
- new net: R13.1, U9.3 (B1)
- new net +VBus: C3.1, C4.1, C5.1, C6.1, P1.A4, P1.A9, P1.B4, P1.B9, U2.1 (VIN), U2.3 (EN), U3.1 (VIN)
- new net SC_FB: R12.2, U3.4 (FB), U9.4 (A)
- new net SC_IO_DIR: U6.5 (DIR)
- new net SC_PWR_EN: R11.1, U3.3 (EN)
- new net SC_PWR_SEL: R15.1, U9.6
- new net SC_RAW_CLK: P2.C3 (CLK), TP_SC3.1, U5.4 (B)
- new net SC_RAW_IO: P2.C7 (IO), TP_SC7.1, U6.4 (B)
- new net SC_RAW_RST: P2.C2 (RST), TP_SC2.1, U4.4 (B)
- new net SC_SW: L2.1, U3.5 (SW)
- new net USB_D+: P1.A6 (D+), P1.B6 (D+)
- new net USB_D-: P1.A7 (D-), P1.B7 (D-)
- new net V_SW: L1.1, U2.5 (SW)
- no-connect marks 0 -> 12
Other:
- moved on the sheet: C10, R10, TP_SC0, TP_SC1, TP_SC2, TP_SC3, TP_SC4, TP_SC5, TP_SC6, TP_SC7, TP_SC8
